File: Nuevos_Modulos/Teclado/Hw/Formant_V2_Teclado.sch (KiCad schematic (older format))
At the start: 13 parts

Commit message: Actualizacion SW Teclado
Parts:
- added D?: 1N4148, symbol D
- added R? (x5): 10K, symbol R
- added SW?: SET CANAL ID, symbol SW_DIP_x04
- added SW?: TEST, symbol SW_Push
- SW?: value PROG -> PROG ARDUINO
Connections:
- wire segments 66 -> 102
Other:
- moved on the sheet: R?
Changed lines of the file:
@@
 L R R?
 U 1 1 595024DD
-P 10000 1250
-F 0 "R?" V 9800 1200 50  0000 C CNN
-F 1 "220" V 9900 1250 50  0000 C CNN
-F 2 "" V 9930 1250 50  0000 C CNN
-F 3 "" H 10000 1250 50  0000 C CNN
-	1    10000 1250
+P 9950 1000
+F 0 "R?" V 9750 950 50  0000 C CNN
+F 1 "220" V 9850 1000 50  0000 C CNN
+F 2 "" V 9880 1000 50  0000 C CNN
+F 3 "" H 9950 1000 50  0000 C CNN
+	1    9950 1000
 	0    1    1    0
 $EndComp
-Wire Wire Line
-	9350 1250 9850 1250
-Text GLabel 10400 1250 2    60   Input ~ 0
+Text GLabel 10350 1000 2    60   Input ~ 0
 MIDI_IN_TX
 Wire Wire Line
-	10150 1250 10400 1250
+	10100 1000 10350 1000
 Text GLabel 10400 1450 2    60   Input ~ 0
 MIDI_IN_GND
@@
 P 7250 1450
 F 0 "SW?" H 7250 1600 50  0000 C CNN
-F 1 "PROG" H 7250 1300 50  0000 C CNN
+F 1 "PROG ARDUINO" H 7250 1300 50  0000 C CNN
 F 2 "" H 7250 1450 50  0000 C CNN
 F 3 "" H 7250 1450 50  0000 C CNN
@@
 Wire Wire Line
 	3800 2950 3900 2950
+$Comp
+L D D?
+U 1 1 5957EDBB
+P 9600 1250
+F 0 "D?" V 9650 1400 50  0000 C CNN
+F 1 "1N4148" V 9550 1500 50  0000 C CNN
+F 2 "" H 9600 1250 50  0000 C CNN
+F 3 "" H 9600 1250 50  0000 C CNN
+	1    9600 1250
+	0    1    1    0
+$EndComp
+Wire Wire Line
+	9800 1000 9400 1000
+Wire Wire Line
+	9400 1000 9400 1250
+Wire Wire Line
+	9400 1250 9350 1250
+Wire Wire Line
+	9600 1100 9600 1000
+Connection ~ 9600 1000
+Wire Wire Line
+	9600 1400 9600 1450
+Connection ~ 9600 1450
+$Comp
+L SW_DIP_x04 SW?
+U 1 1 5957FAC3
+P 6400 4700
+F 0 "SW?" V 6400 5100 50  0000 C CNN
+F 1 "SET CANAL ID" V 6300 5300 50  0000 C CNN
+F 2 "" H 6400 4700 50  0000 C CNN
+F 3 "" H 6400 4700 50  0000 C CNN
+	1    6400 4700
+	0    1    1    0
+$EndComp
+$Comp
+L R R?
+U 1 1 5957FC1B
+P 6300 4050
+F 0 "R?" V 6350 4200 50  0000 C CNN
+F 1 "10K" V 6300 4050 50  0000 C CNN
+F 2 "" V 6230 4050 50  0000 C CNN
+F 3 "" H 6300 4050 50  0000 C CNN
+	1    6300 4050
+	-1   0    0    1
+$EndComp
+$Comp
+L R R?
+U 1 1 5957FCB5
+P 6400 4050
+F 0 "R?" V 6450 4200 50  0000 C CNN
+F 1 "10K" V 6400 4050 50  0000 C CNN
+F 2 "" V 6330 4050 50  0000 C CNN
+F 3 "" H 6400 4050 50  0000 C CNN
+	1    6400 4050
+	-1   0    0    1
+$EndComp
+Wire Wire Line
+	6300 4200 6300 4400
+Wire Wire Line
+	6400 4200 6400 4400
+$Comp
+L R R?
+U 1 1 59580225
+P 6500 4050
+F 0 "R?" V 6550 4200 50  0000 C CNN
+F 1 "10K" V 6500 4050 50  0000 C CNN
+F 2 "" V 6430 4050 50  0000 C CNN
+F 3 "" H 6500 4050 50  0000 C CNN
+	1    6500 4050
+	-1   0    0    1
+$EndComp
+$Comp
+L R R?
+U 1 1 5958022B
+P 6600 4050
+F 0 "R?" V 6650 4200 50  0000 C CNN
+F 1 "10K" V 6600 4050 50  0000 C CNN
+F 2 "" V 6530 4050 50  0000 C CNN
+F 3 "" H 6600 4050 50  0000 C CNN
+	1    6600 4050
+	-1   0    0    1
+$EndComp
+Wire Wire Line
+	6500 4200 6500 4400
+Wire Wire Line
+	6600 4200 6600 4400
+$Comp
+L GND #PWR?
+U 1 1 5958026E
+P 6600 5200
+F 0 "#PWR?" H 6600 4950 50  0001 C CNN
+F 1 "GND" H 6600 5050 50  0000 C CNN
+F 2 "" H 6600 5200 50  0000 C CNN
+F 3 "" H 6600 5200 50  0000 C CNN
+	1    6600 5200
+	1    0    0    -1
+$EndComp
+Wire Wire Line
+	6600 5000 6600 5200
+Wire Wire Line
+	6300 5000 6300 5150
+Wire Wire Line
+	5550 5150 6600 5150
+Connection ~ 6600 5150
+Wire Wire Line
+	6400 5000 6400 5150
+Connection ~ 6400 5150
+Wire Wire Line
+	6500 5000 6500 5150
+Connection ~ 6500 5150
+$Comp
+L +5V #PWR?
+U 1 1 59580882
+P 6600 3750
+F 0 "#PWR?" H 6600 3600 50  0001 C CNN
+F 1 "+5V" H 6600 3890 50  0000 C CNN
+F 2 "" H 6600 3750 50  0000 C CNN
+F 3 "" H 6600 3750 50  0000 C CNN
+	1    6600 3750
+	1    0    0    -1
+$EndComp
+Wire Wire Line
+	6600 3750 6600 3900
+Wire Wire Line
+	6600 3800 6300 3800
+Wire Wire Line
+	6300 3800 6300 3900
+Connection ~ 6600 3800
+Wire Wire Line
+	6400 3900 6400 3800
+Connection ~ 6400 3800
+Wire Wire Line
+	6500 3800 6500 3900
+Connection ~ 6500 3800
+Wire Wire Line
+	5100 3550 6200 3550
+Wire Wire Line
+	6200 3550 6200 4250
+Wire Wire Line
+	6200 4250 6600 4250
+Connection ~ 6600 4250
+Wire Wire Line
+	5100 3650 6150 3650
+Wire Wire Line
+	6150 3650 6150 4300
+Wire Wire Line
+	5100 3750 6100 3750
+Wire Wire Line
+	6100 3750 6100 4350
+Wire Wire Line
+	6150 4300 6500 4300
+Connection ~ 6500 4300
+Wire Wire Line
+	6100 4350 6400 4350
+Connection ~ 6400 4350
+Wire Wire Line
+	5100 3850 6050 3850
+Wire Wire Line
+	6050 3850 6050 4400
+Wire Wire Line
+	6050 4400 6300 4400
+Connection ~ 6300 4400
+$Comp
+L SW_Push SW?
+U 1 1 59581257
+P 5550 4700
+F 0 "SW?" V 5500 4500 50  0000 L CNN
+F 1 "TEST" V 5400 4550 50  0000 C CNN
+F 2 "" H 5550 4900 50  0000 C CNN
+F 3 "" H 5550 4900 50  0000 C CNN
+	1    5550 4700
+	0    1    1    0
+$EndComp
+Wire Wire Line
+	5550 4900 5550 5150
+Connection ~ 6300 5150
+$Comp
+L R R?
+U 1 1 595814A4
+P 5550 4250
+F 0 "R?" H 5450 4300 50  0000 C CNN
+F 1 "10K" H 5400 4200 50  0000 C CNN
+F 2 "" V 5480 4250 50  0000 C CNN
+F 3 "" H 5550 4250 50  0000 C CNN
+	1    5550 4250
+	-1   0    0    1
+$EndComp
+$Comp
+L +5V #PWR?
+U 1 1 595815EC
+P 5550 4050
+F 0 "#PWR?" H 5550 3900 50  0001 C CNN
+F 1 "+5V" H 5550 4190 50  0000 C CNN
+F 2 "" H 5550 4050 50  0000 C CNN
+F 3 "" H 5550 4050 50  0000 C CNN
+	1    5550 4050
+	1    0    0    -1
+$EndComp
+Wire Wire Line
+	5550 4050 5550 4100
+Wire Wire Line
+	5550 4400 5550 4500
+Wire Wire Line
+	5550 4450 5350 4450
+Wire Wire Line
+	5350 4450 5350 3950
+Wire Wire Line
+	5350 3950 5100 3950
+Connection ~ 5550 4450
 $EndSCHEMATC

Commit message: Actualizacion HW
Parts:
- added C?: 1nF, symbol C_Small
- added R? (x54): 100, symbol R
- added R?: 3K3, symbol R
- added R?: 750, symbol R
- added R?: 13K7, symbol R
- added RV?: 4K7, symbol POT_TRIM
- added U?: 74HCT138, symbol 74LS138
- added U?: LF356, symbol LM741
- added U? (x7): 4051, symbol 4051
- added U?: LM741, symbol LM741
- SW?: value SET CANAL ID -> SET CANAL MIDI ID
Connections:
- net labels added: +15V, -15V, KBV
- wire segments 102 -> 421
Other:
- moved on the sheet: ARDUINO?, D?, R?, SW?, U?, U?A, U?B
