File: Nuevos_Modulos/Teclado/Hw/Formant_V2_Teclado.sch (KiCad schematic (older format))
At the start: 90 parts

Commit message: Informacion COM
Parts:
- added C?: 100nF, symbol C_Small
- added R? (x3): 100K, symbol R
- added RV?: COM Volumen, symbol POT
Connections:
- net +5V: now also RV?.1
- net GND: now also C?.1, R?.1, R?.1, R?.1, RV?.3
- net at ARDUINO?.19 (A0): now also C?.2, RV?.2
- net COM_VOL_DATA: now reaches ARDUINO?.20 (A1)
- net COM_VOL_RESET: now reaches ARDUINO?.21 (A2)
- net COM_VOL_RESET: now also R?.2
- net COM_VOL_CLOCK: now reaches ARDUINO?.22 (A3)
- net COM_VOL_CLOCK: now also R?.2
Changed lines of the file:
@@
 LIBS:arduino
 LIBS:switches
+LIBS:Baphomet_Libreria
 LIBS:Formant_V2_Teclado-cache
 EELAYER 25 0
@@
 	1075 1250 1075 775
 Connection ~ 1075 775
+$Comp
+L POT RV?
+U 1 1 599497D0
+P 7500 8275
+F 0 "RV?" H 7900 8425 50  0000 C CNN
+F 1 "COM Volumen" H 8075 8350 50  0000 C CNN
+F 2 "" H 7500 8275 50  0000 C CNN
+F 3 "" H 7500 8275 50  0000 C CNN
+	1    7500 8275
+	1    0    0    -1
+$EndComp
+Wire Wire Line
+	7950 7400 7750 7400
+Wire Wire Line
+	7750 7400 7750 8325
+Wire Wire Line
+	7750 8275 7650 8275
+$Comp
+L GND #PWR?
+U 1 1 59949BFE
+P 7500 8550
+F 0 "#PWR?" H 7500 8300 50  0001 C CNN
+F 1 "GND" H 7500 8400 50  0000 C CNN
+F 2 "" H 7500 8550 50  0000 C CNN
+F 3 "" H 7500 8550 50  0000 C CNN
+	1    7500 8550
+	1    0    0    -1
+$EndComp
+Wire Wire Line
+	7500 8425 7500 8550
+$Comp
+L +5V #PWR?
+U 1 1 5994A5AB
+P 7500 8025
+F 0 "#PWR?" H 7500 7875 50  0001 C CNN
+F 1 "+5V" H 7500 8165 50  0000 C CNN
+F 2 "" H 7500 8025 50  0000 C CNN
+F 3 "" H 7500 8025 50  0000 C CNN
+	1    7500 8025
+	1    0    0    -1
+$EndComp
+Wire Wire Line
+	7500 8025 7500 8125
+Text GLabel 6900 7300 0    60   Output ~ 0
+COM_VOL_DATA
+Wire Wire Line
+	6900 7300 7950 7300
+Text GLabel 6900 7200 0    60   Output ~ 0
+COM_VOL_RESET
+Wire Wire Line
+	6900 7200 7950 7200
+Text GLabel 6900 7100 0    60   Output ~ 0
+COM_VOL_CLOCK
+Wire Wire Line
+	6900 7100 7950 7100
+$Comp
+L R R?
+U 1 1 5994F6D2
+P 7250 8275
+F 0 "R?" V 7300 8425 50  0000 C CNN
+F 1 "100K" V 7250 8275 50  0000 C CNN
+F 2 "" V 7180 8275 50  0000 C CNN
+F 3 "" H 7250 8275 50  0000 C CNN
+	1    7250 8275
+	-1   0    0    1
+$EndComp
+$Comp
+L R R?
+U 1 1 5994F842
+P 7100 8275
+F 0 "R?" V 7150 8425 50  0000 C CNN
+F 1 "100K" V 7100 8275 50  0000 C CNN
+F 2 "" V 7030 8275 50  0000 C CNN
+F 3 "" H 7100 8275 50  0000 C CNN
+	1    7100 8275
+	-1   0    0    1
+$EndComp
+$Comp
+L R R?
+U 1 1 5994F9A3
+P 6950 8275
+F 0 "R?" V 7000 8425 50  0000 C CNN
+F 1 "100K" V 6950 8275 50  0000 C CNN
+F 2 "" V 6880 8275 50  0000 C CNN
+F 3 "" H 6950 8275 50  0000 C CNN
+	1    6950 8275
+	-1   0    0    1
+$EndComp
+Wire Wire Line
+	6950 8425 6950 8550
+Wire Wire Line
+	6950 8550 7750 8550
+Wire Wire Line
+	7100 8425 7100 8550
+Connection ~ 7100 8550
+Wire Wire Line
+	7250 8425 7250 8550
+Connection ~ 7250 8550
+Connection ~ 7500 8550
+Wire Wire Line
+	7250 8100 7250 7300
+Connection ~ 7250 7300
+Wire Wire Line
+	7100 8125 7100 7200
+Connection ~ 7100 7200
+Wire Wire Line
+	6950 7100 6950 8125
+Connection ~ 6950 7100
+$Comp
+L C_Small C?
+U 1 1 59956A1E
+P 7750 8425
+F 0 "C?" V 7600 8475 50  0000 L CNN
+F 1 "100nF" H 7400 8425 50  0000 L CNN
+F 2 "" H 7750 8425 50  0000 C CNN
+F 3 "" H 7750 8425 50  0000 C CNN
+	1    7750 8425
+	-1   0    0    1
+$EndComp
+Wire Wire Line
+	7750 8550 7750 8525
+Connection ~ 7750 8275
 $EndSCHEMATC

Commit message: Actualizacion SW MIDI Volumen
Parts:
- removed R? (x3): 100K, symbol R
Changed lines of the file:
@@
 Wire Wire Line
 	6900 7100 7950 7100
-$Comp
-L R R?
-U 1 1 5994F6D2
-P 7250 8275
-F 0 "R?" V 7300 8425 50  0000 C CNN
-F 1 "100K" V 7250 8275 50  0000 C CNN
-F 2 "" V 7180 8275 50  0000 C CNN
-F 3 "" H 7250 8275 50  0000 C CNN
-	1    7250 8275
-	-1   0    0    1
-$EndComp
-$Comp
-L R R?
-U 1 1 5994F842
-P 7100 8275
-F 0 "R?" V 7150 8425 50  0000 C CNN
-F 1 "100K" V 7100 8275 50  0000 C CNN
-F 2 "" V 7030 8275 50  0000 C CNN
-F 3 "" H 7100 8275 50  0000 C CNN
-	1    7100 8275
-	-1   0    0    1
-$EndComp
-$Comp
-L R R?
-U 1 1 5994F9A3
-P 6950 8275
-F 0 "R?" V 7000 8425 50  0000 C CNN
-F 1 "100K" V 6950 8275 50  0000 C CNN
-F 2 "" V 6880 8275 50  0000 C CNN
-F 3 "" H 6950 8275 50  0000 C CNN
-	1    6950 8275
-	-1   0    0    1
-$EndComp
-Wire Wire Line
-	6950 8425 6950 8550
-Wire Wire Line
-	6950 8550 7750 8550
-Wire Wire Line
-	7100 8425 7100 8550
-Connection ~ 7100 8550
-Wire Wire Line
-	7250 8425 7250 8550
-Connection ~ 7250 8550
 Connection ~ 7500 8550
-Wire Wire Line
-	7250 8100 7250 7300
-Connection ~ 7250 7300
-Wire Wire Line
-	7100 8125 7100 7200
-Connection ~ 7100 7200
-Wire Wire Line
-	6950 7100 6950 8125
-Connection ~ 6950 7100
 $Comp
 L C_Small C?
@@
 	7750 8550 7750 8525
 Connection ~ 7750 8275
+Wire Wire Line
+	7500 8550 7750 8550
 $EndSCHEMATC

Commit message: Actualizacion DOC
Parts:
- added 10uF/16v: CP, symbol CP
- added C?: 220nF, symbol C_Small
- added C?: 680nF, symbol C_Small
- added D?: 1N4148, symbol D
- added Q? (x3): BF256B, TO-92, symbol BF245B
- added R?: 10K, symbol R
- added R? (x2): 1K, symbol R
- added R? (x2): 12K 1%, symbol R
- added R?: 1M, symbol R
- added RV?: POT, symbol POT
Connections:
- net +15V: now also Q?.3 (D), Q?.3 (D)
- net +5V: now also C?.2
- net -15V: now also R?.2, R?.2
- net GND: now also 10uF/16v.2, C?.1, C?.1
- net KBV: now also R?.1
- new net: R?.1, RV?.2
- new net: C?.2, Q?.1 (G), R?.2
- new net: Q?.2 (S), Q?.2 (S), R?.1, R?.1
- new net: D?.2 (A), Q?.1 (G), R?.2
- new net: C?.2, Q?.1 (G), Q?.3 (D)
- new net: Q?.2 (S), R?.1, R?.2
- new net: R?.1, RV?.2, RV?.3
- new net POT_VOL_MANUAL: 10uF/16v.1, ARDUINO?.19 (A0), R?.2
Other:
- moved on the sheet: ARDUINO?, C?, D?, R?, RV?, SW?, U?, U?A, U?B

Commit message: Actualizacion Hw
Parts:
- RV?: value COM Volumen -> 10K
Connections:
- net RESET_GENERAL: now reaches ARDUINO?.28 (RST)
Other:
- note added: "Esta montado en el módulo COM"
- moved on the sheet: 10uF/16v, C?, R?, RV?
Changed lines of the file:
@@
 L GND #PWR?
 U 1 1 59502305
-P 7650 7600
-F 0 "#PWR?" H 7650 7350 50  0001 C CNN
-F 1 "GND" H 7650 7450 50  0000 C CNN
-F 2 "" H 7650 7600 50  0000 C CNN
-F 3 "" H 7650 7600 50  0000 C CNN
-	1    7650 7600
-	1    0    0    -1
+P 7650 7250
+F 0 "#PWR?" H 7650 7000 50  0001 C CNN
+F 1 "GND" H 7650 7100 50  0000 C CNN
+F 2 "" H 7650 7250 50  0000 C CNN
+F 3 "" H 7650 7250 50  0000 C CNN
+	1    7650 7250
+	-1   0    0    1
 $EndComp
 Wire Wire Line
@@
 	9900 7400 9500 7400
 Wire Wire Line
-	9500 7400 9500 8000
+	9500 6900 9500 8000
 Wire Wire Line
 	9400 7150 9400 7900
@@
 L POT RV?
 U 1 1 599497D0
-P 6525 9450
-F 0 "RV?" H 6150 9200 50  0000 C CNN
-F 1 "COM Volumen" H 5950 9300 50  0000 C CNN
-F 2 "" H 6525 9450 50  0000 C CNN
-F 3 "" H 6525 9450 50  0000 C CNN
-	1    6525 9450
+P 7125 10150
+F 0 "RV?" H 7250 9900 50  0000 C CNN
+F 1 "10K" H 7250 10000 50  0000 C CNN
+F 2 "" H 7125 10150 50  0000 C CNN
+F 3 "" H 7125 10150 50  0000 C CNN
+	1    7125 10150
 	1    0    0    -1
 $EndComp
@@
 L GND #PWR?
 U 1 1 59949BFE
-P 6525 9925
-F 0 "#PWR?" H 6525 9675 50  0001 C CNN
-F 1 "GND" H 6525 9775 50  0000 C CNN
-F 2 "" H 6525 9925 50  0000 C CNN
-F 3 "" H 6525 9925 50  0000 C CNN
-	1    6525 9925
-	1    0    0    -1
-$EndComp
-Wire Wire Line
-	6525 9600 6525 9925
+P 7125 10625
+F 0 "#PWR?" H 7125 10375 50  0001 C CNN
+F 1 "GND" H 7125 10475 50  0000 C CNN
+F 2 "" H 7125 10625 50  0000 C CNN
+F 3 "" H 7125 10625 50  0000 C CNN
+	1    7125 10625
+	1    0    0    -1
+$EndComp
+Wire Wire Line
+	7125 10300 7125 10625
 $Comp
 L +5V #PWR?
 U 1 1 5994A5AB
-P 6525 9200
-F 0 "#PWR?" H 6525 9050 50  0001 C CNN
-F 1 "+5V" H 6525 9340 50  0000 C CNN
-F 2 "" H 6525 9200 50  0000 C CNN
-F 3 "" H 6525 9200 50  0000 C CNN
-	1    6525 9200
-	1    0    0    -1
-$EndComp
-Wire Wire Line
-	6525 9200 6525 9300
+P 7125 9900
+F 0 "#PWR?" H 7125 9750 50  0001 C CNN
+F 1 "+5V" H 7125 10040 50  0000 C CNN
+F 2 "" H 7125 9900 50  0000 C CNN
+F 3 "" H 7125 9900 50  0000 C CNN
+	1    7125 9900
+	1    0    0    -1
+$EndComp
+Wire Wire Line
+	7125 9900 7125 10000
 Text GLabel 6950 8500 0    60   Output ~ 0
 COM_VOL_DATA
@@
 Wire Wire Line
 	6950 8300 8000 8300
-Connection ~ 6525 9725
+Connection ~ 7125 10425
 $Comp
 L C_Small C?
 U 1 1 59956A1E
-P 6250 9450
-F 0 "C?" H 6425 9475 50  0000 L CNN
-F 1 "100nF" H 6400 9375 50  0000 L CNN
-F 2 "" H 6250 9450 50  0000 C CNN
-F 3 "" H 6250 9450 50  0000 C CNN
-	1    6250 9450
+P 6850 10150
+F 0 "C?" H 7025 10175 50  0000 L CNN
+F 1 "100nF" H 7000 10075 50  0000 L CNN
+F 2 "" H 6850 10150 50  0000 C CNN
+F 3 "" H 6850 10150 50  0000 C CNN
+	1    6850 10150
 	-1   0    0    1
 $EndComp
 Wire Wire Line
-	6525 9725 6250 9725
-Wire Wire Line
-	6250 9725 6250 9550
-Wire Wire Line
-	6250 9350 6250 9250
-Wire Wire Line
-	6250 9250 6525 9250
-Connection ~ 6525 9250
+	7125 10425 6850 10425
+Wire Wire Line
+	6850 10425 6850 10250
+Wire Wire Line
+	6850 10050 6850 9950
+Wire Wire Line
+	6850 9950 7125 9950
+Connection ~ 7125 9950
 $Comp
 L R R?
 U 1 1 5996C374
-P 6900 9450
-F 0 "R?" V 6975 9525 50  0000 C CNN
-F 1 "10K" V 7075 9500 50  0000 C CNN
-F 2 "" V 6830 9450 50  0000 C CNN
-F 3 "" H 6900 9450 50  0000 C CNN
-	1    6900 9450
+P 7500 10150
+F 0 "R?" V 7575 10225 50  0000 C CNN
+F 1 "10K" V 7675 10200 50  0000 C CNN
+F 2 "" V 7430 10150 50  0000 C CNN
+F 3 "" H 7500 10150 50  0000 C CNN
+	1    7500 10150
 	0    -1   -1   0
 $EndComp
 Wire Wire Line
-	6675 9450 6750 9450
-Wire Wire Line
-	7050 9450 7350 9450
+	7275 10150 7350 10150
+Wire Wire Line
+	7650 10150 7950 10150
 $Comp
 L CP 10uF/16v
 U 1 1 5996D0DD
-P 7125 9650
-F 0 "10uF/16v" H 7150 9750 50  0000 L CNN
-F 1 "CP" H 7150 9550 50  0000 L CNN
-F 2 "" H 7163 9500 50  0000 C CNN
-F 3 "" H 7125 9650 50  0000 C CNN
-	1    7125 9650
-	1    0    0    -1
-$EndComp
-Connection ~ 7125 9450
+P 7725 10350
+F 0 "10uF/16v" H 7900 10350 50  0000 L CNN
+F 1 "CP" H 7750 10250 50  0000 L CNN
+F 2 "" H 7763 10200 50  0000 C CNN
+F 3 "" H 7725 10350 50  0000 C CNN
+	1    7725 10350
+	1    0    0    -1
+$EndComp
+Connection ~ 7725 10150
 $Comp
 L GND #PWR?
 U 1 1 5996EB06
-P 7125 9925
-F 0 "#PWR?" H 7125 9675 50  0001 C CNN
-F 1 "GND" H 7125 9775 50  0000 C CNN
-F 2 "" H 7125 9925 50  0000 C CNN
-F 3 "" H 7125 9925 50  0000 C CNN
-	1    7125 9925
-	1    0    0    -1
-$EndComp
-Wire Wire Line
-	7125 9800 7125 9925
-Text GLabel 7350 9450 2    60   Output ~ 0
+P 7725 10625
+F 0 "#PWR?" H 7725 10375 50  0001 C CNN
+F 1 "GND" H 7725 10475 50  0000 C CNN
+F 2 "" H 7725 10625 50  0000 C CNN
+F 3 "" H 7725 10625 50  0000 C CNN
+	1    7725 10625
+	1    0    0    -1
+$EndComp
+Wire Wire Line
+	7725 10500 7725 10625
+Text GLabel 7950 10150 2    60   Output ~ 0
 POT_VOL_MANUAL
 Wire Wire Line
-	7125 9450 7125 9500
+	7725 10150 7725 10200
 Text GLabel 6950 8725 0    60   Input ~ 0
 POT_VOL_MANUAL
@@
 	11925 3050 11925 3000
 Connection ~ 11700 2850
+Wire Notes Line
+	6500 9600 9000 9600
+Wire Notes Line
+	9000 9600 9000 11100
+Wire Notes Line
+	9000 11100 6400 11100
+Wire Notes Line
+	6400 11100 6400 9600
+Wire Notes Line
+	6400 9600 6750 9600
+Text Notes 7400 11000 0    60   ~ 0
+Esta montado en el módulo COM
+Text GLabel 6900 7700 0    60   Input ~ 0
+RESET_GENERAL
+Wire Wire Line
+	8000 7700 6900 7700
+Wire Wire Line
+	7650 7600 7650 7250
+Text GLabel 10500 6900 0    60   Output ~ 0
+LED_SEÑAL_MIDI
+Wire Wire Line
+	9750 6900 9500 6900
+Connection ~ 9500 7400
 $EndSCHEMATC

Commit message: Actualizacion HW Teclado
Parts:
- removed C?: 220nF, symbol C_Small
- removed Q?: BF256B, TO-92, symbol BF245B
- removed R?: 12K 1%, symbol R
- removed R?: 1M, symbol R
- removed RV?: POT, symbol POT
- added C?: 680nF, symbol C_Small
- added C? (x2): 220nF, symbol C_Small
- added C?: 22nF, symbol C_Small
- added D?: 1N4148, symbol D
- added Q? (x2): BF256B, TO-92, symbol BF245B
- added R? (x2): *12K 1%, symbol R
- added R? (x4): *100K, symbol R
- added R?: 300K, symbol R
- added R?: 15K, symbol R
- added R? (x2): 47K, symbol R
- added R?: 1M, symbol R
- added R? (x2): 100K, symbol R
- added R?: 12K, symbol R
- added R?: 2K2, symbol R
- added R?: 1K, symbol R
- added R?: 10K, symbol R
- added R?: 100ohm, symbol R
- added RV?: 1M Log, symbol POT
- added RV?: 100K Lin, symbol POT
- added RV?: 100K, symbol POT_TRIM
- added RV?: *100K, symbol POT_TRIM
- added RV? (x2): 100K Log, symbol POT
- added SW?: S1, symbol SW_DPDT_x2
- added U? (x4): LM741, symbol LM741
- R?: value 12K 1% -> *12K 1%
Connections:
- net +15V: now also Q?.3 (D), Q?.3 (D), R?.1, R?.2, RV?.1, U?.7 (V+), U?.7 (V+), U?.7 (V+), U?.7 (V+)
- net -15V: now also R?.2, R?.2, RV?.1, RV?.3, U?.4 (V-), U?.4 (V-), U?.4 (V-), U?.4 (V-)
- net GND: now also C?.1, C?.1, C?.1, C?.1, R?.1, R?.2, R?.2, R?.2, R?.2, RV?.1, RV?.3, RV?.3, SW?.1 (A)
- net PUNTO_E: now also C?.2, R?.1, U?.3 (+)
- net at R?.2: now also C?.2, Q?.1 (G)
- net at Q?.2 (S): now also Q?.2 (S), R?.1, R?.1
- net at D?.2 (A), Q?.1 (G): now also R?.2
- net at D?.1 (K): now also R?.2, U?.6
- net at R?.1: now also RV?.2, RV?.3
- new net: C?.2, Q?.1 (G), RV?.1
- new net: Q?.2 (S), R?.1, R?.2
- new net: R?.1, R?.1, R?.1, R?.1, R?.2, R?.2, U?.2 (-)
- new net: R?.2, SW?.2 (B)
- new net: R?.1, U?.3 (+) (x2)
- new net: R?.1, R?.2, U?.6
- new net: R?.1, U?.2 (-)
- new net: RV?.2, SW?.3 (C)
- new net: D?.1 (K), RV?.3, U?.2 (-), U?.6
- new net: C?.2, D?.2 (A), RV?.1, RV?.2, U?.3 (+)
- new net: R?.1, R?.2, U?.2 (-)
- new net: R?.2, RV?.2 (x2)
- new net: R?.1, RV?.2
- new net: R?.1, R?.2, RV?.3
- new net FM: RV?.1
- new net GATE: R?.1
- new net KOV: U?.6
Other:
- note added: "2V3->"
- moved on the sheet: C?, D?, Q?, R?

Commit message: Actualizacion Documentacion
Parts:
- removed R?: 10K, symbol R
- removed U? (x4): LM741, symbol LM741
- added R?: *100K, symbol R
- added U?: DS1801, symbol DS1801
- added U? (x4): LM358, symbol LM358
Connections:
- net +15V: now also U?.4 (V-), U?.4 (V-), U?.8 (V+), U?.8 (V+)
- net +5V: now also U?.14 (VCC)
- net -15V: now also U?.4 (V-), U?.4 (V-), U?.8 (V+), U?.8 (V+)
- net GND: now also U?.1 (GND), U?.11 (AGND), U?.6 (L0), U?.9 (L1)
- net KOV: now also R?.1, U?.1
- net PUNTO_E: now also U?.3 (+)
- net at R?.1, R?.1, R?.1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: now also U?.6 (-)
- net at R?.1: now also U?.5 (+)
- net at R?.1, R?.2: now also U?.7
- net at R?.1: now also R?.2, U?.2 (-)
- net at R?.1: now also U?.3 (+)
- net at D?.1 (K), R?.2: now also U?.7
- net at D?.1 (K), RV?.3: now also U?.1, U?.2 (-)
- net at C?.2, D?.2 (A), RV?.1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: now also U?.5 (+)
- net at R?.1, R?.2: now also U?.6 (-)
- net COM_VOL_CLOCK: no longer names the net of ARDUINO?.22 (A3)
- net COM_VOL_CLOCK: now also U?.13 (CLK)
- net COM_VOL_DATA: no longer names the net of ARDUINO?.20 (A1)
- net COM_VOL_DATA: now also U?.12 (D)
- net COM_VOL_RESET: no longer names the net of ARDUINO?.21 (A2)
- net COM_VOL_RESET: now also U?.3 (RST)
- new net POT_1a_CUR: U?.8 (W1)
- new net POT_1a_ENT: U?.10 (H1)
- new net POT_1b_CUR: U?.5 (W0)
- new net POT_1b_ENT: U?.7 (H0)
Other:
- moved on the sheet: 10uF/16v, C?, R?, RV?

Commit message: Actualizacion DOC/HW
Parts:
- removed R? (x6): 100, symbol R
- removed R?: 750, symbol R
- added R?: 100K, symbol R
- added R?: 750, symbol R
Connections:
- net GND: now also U?.1 (X4), U?.12 (X3), U?.15 (X2), U?.2 (X6), U?.4 (X7), U?.5 (X5), R?.2
- net POT_VOL_MANUAL: now also R?.1
- net at C?.2, R?.2, U?.2 (-): now also R?.2
- net at R?.2, U?.14 (X1): now also R?.1
Other:
- moved on the sheet: C?, R?, RV?
Changed lines of the file:
@@
 L C_Small C?
 U 1 1 598FD58E
-P 2025 775
-F 0 "C?" V 1875 825 50  0000 L CNN
-F 1 "1nF" V 1950 825 50  0000 L CNN
-F 2 "" H 2025 775 50  0000 C CNN
-F 3 "" H 2025 775 50  0000 C CNN
-	1    2025 775
-	0    1    1    0
-$EndComp
-Wire Wire Line
-	2125 775  2225 775
-Wire Wire Line
-	2225 775  2225 1100
+P 2100 800
+F 0 "C?" V 1950 850 50  0000 L CNN
+F 1 "1nF" V 2025 850 50  0000 L CNN
+F 2 "" H 2100 800 50  0000 C CNN
+F 3 "" H 2100 800 50  0000 C CNN
+	1    2100 800
+	0    1    1    0
+$EndComp
 Wire Wire Line
 	2125 1100 3750 1100
-Wire Wire Line
-	725  775  1925 775
 $Comp
 L +15V #PWR?
@@
 	1    0    0    -1
 $EndComp
-$Comp
-L R R?
-U 1 1 599012B2
-P 3525 9700
-F 0 "R?" V 3475 9475 50  0000 C CNN
-F 1 "100" V 3425 9700 50  0000 C CNN
-F 2 "" V 3455 9700 50  0000 C CNN
-F 3 "" H 3525 9700 50  0000 C CNN
-	1    3525 9700
-	0    1    1    0
-$EndComp
-$Comp
-L R R?
-U 1 1 599012B8
-P 3525 9800
-F 0 "R?" V 3475 9575 50  0000 C CNN
-F 1 "100" V 3625 9800 50  0000 C CNN
-F 2 "" V 3455 9800 50  0000 C CNN
-F 3 "" H 3525 9800 50  0000 C CNN
-	1    3525 9800
-	0    1    1    0
-$EndComp
-$Comp
-L R R?
-U 1 1 599012BE
-P 3525 9900
-F 0 "R?" V 3475 9675 50  0000 C CNN
-F 1 "100" V 3425 9900 50  0000 C CNN
-F 2 "" V 3455 9900 50  0000 C CNN
-F 3 "" H 3525 9900 50  0000 C CNN
-	1    3525 9900
-	0    1    1    0
-$EndComp
-Wire Wire Line
-	3375 9600 3375 9650
-Wire Wire Line
-	3675 9700 3850 9700
-Wire Wire Line
-	3375 9700 3375 9750
-Wire Wire Line
-	3675 9800 3850 9800
-Wire Wire Line
-	3375 9650 3750 9650
-Wire Wire Line
-	3750 9650 3750 9700
-Connection ~ 3750 9700
-Wire Wire Line
-	3375 9750 3750 9750
-Wire Wire Line
-	3750 9750 3750 9800
-Connection ~ 3750 9800
-Wire Wire Line
-	3675 9900 3850 9900
-Wire Wire Line
-	3375 9800 3375 9850
-Wire Wire Line
-	3375 9850 3750 9850
-Wire Wire Line
-	3750 9850 3750 9900
-Connection ~ 3750 9900
-$Comp
-L R R?
-U 1 1 599012D4
-P 3525 10000
-F 0 "R?" V 3475 9775 50  0000 C CNN
-F 1 "100" V 3625 10000 50  0000 C CNN
-F 2 "" V 3455 10000 50  0000 C CNN
-F 3 "" H 3525 10000 50  0000 C CNN
-	1    3525 10000
-	0    1    1    0
-$EndComp
-$Comp
-L R R?
-U 1 1 599012DA
-P 3525 10100
-F 0 "R?" V 3475 9875 50  0000 C CNN
-F 1 "100" V 3425 10100 50  0000 C CNN
-F 2 "" V 3455 10100 50  0000 C CNN
-F 3 "" H 3525 10100 50  0000 C CNN
-	1    3525 10100
-	0    1    1    0
-$EndComp
-Wire Wire Line
-	3675 10000 3850 10000
-Wire Wire Line
-	3675 10100 3850 10100
-$Comp
-L R R?
-U 1 1 599012E9
-P 3525 9600
-F 0 "R?" V 3475 9375 50  0000 C CNN
-F 1 "100" V 3625 9600 50  0000 C CNN
-F 2 "" V 3455 9600 50  0000 C CNN
-F 3 "" H 3525 9600 50  0000 C CNN
-	1    3525 9600
-	0    1    1    0
-$EndComp
-Wire Wire Line
-	3375 9900 3375 9950
-Wire Wire Line
-	3375 9950 3750 9950
-Wire Wire Line
-	3750 9950 3750 10000
-Connection ~ 3750 10000
-Wire Wire Line
-	3375 10000 3375 10050
-Wire Wire Line
-	3375 10050 3750 10050
-Wire Wire Line
-	3750 10050 3750 10100
-Connection ~ 3750 10100
-Wire Wire Line
-	3375 10100 3375 10200
 Connection ~ 3750 9600
 Wire Wire Line
@@
 Wire Wire Line
 	1400 1000 1400 1250
-Wire Wire Line
-	1525 1200 1475 1200
-Wire Wire Line
-	1475 1200 1475 775
 $Comp
 L GND #PWR?
@@
 $Comp
 L R R?
-U 1 1 599161D3
-P 1075 1400
-F 0 "R?" H 1225 1500 50  0000 C CNN
-F 1 "750" H 1225 1400 50  0000 C CNN
-F 2 "" V 1005 1400 50  0000 C CNN
-F 3 "" H 1075 1400 50  0000 C CNN
-	1    1075 1400
-	-1   0    0    1
-$EndComp
-$Comp
-L R R?
 U 1 1 59916345
-P 725 1400
-F 0 "R?" H 875 1500 50  0000 C CNN
-F 1 "13K7" H 875 1400 50  0000 C CNN
-F 2 "" V 655 1400 50  0000 C CNN
-F 3 "" H 725 1400 50  0000 C CNN
-	1    725  1400
+P 750 1425
+F 0 "R?" H 900 1525 50  0000 C CNN
+F 1 "13K7" H 900 1425 50  0000 C CNN
+F 2 "" V 680 1425 50  0000 C CNN
+F 3 "" H 750 1425 50  0000 C CNN
+	1    750  1425
 	-1   0    0    1
 $EndComp
@@
 L POT_TRIM RV?
 U 1 1 59917954
-P 725 1825
-F 0 "RV?" V 550 1825 50  0000 C CNN
-F 1 "4K7" V 625 1825 50  0000 C CNN
-F 2 "" H 725 1825 50  0000 C CNN
-F 3 "" H 725 1825 50  0000 C CNN
-	1    725  1825
-	1    0    0    -1
-$EndComp
-Wire Wire Line
-	725  1550 725  1675
-Wire Wire Line
-	725  1975 725  2225
-Wire Wire Line
-	725  2125 875  2125
-Wire Wire Line
-	875  2125 875  1825
+P 750 1850
+F 0 "RV?" V 575 1850 50  0000 C CNN
+F 1 "4K7" V 650 1850 50  0000 C CNN
+F 2 "" H 750 1850 50  0000 C CNN
+F 3 "" H 750 1850 50  0000 C CNN
+	1    750  1850
+	1    0    0    -1
+$EndComp
+Wire Wire Line
+	750  1575 750  1700
+Wire Wire Line
+	750  2000 750  2250
+Wire Wire Line
+	750  2150 900  2150
+Wire Wire Line
+	900  2150 900  1850
 $Comp
 L -15V #PWR?
 U 1 1 59918EFC
-P 725 2225
-F 0 "#PWR?" H 725 2325 50  0001 C CNN
-F 1 "-15V" H 725 2375 50  0000 C CNN
-F 2 "" H 725 2225 50  0000 C CNN
-F 3 "" H 725 2225 50  0000 C CNN
-	1    725  2225
-	-1   0    0    1
-$EndComp
-Connection ~ 725  2125
+P 750 2250
+F 0 "#PWR?" H 750 2350 50  0001 C CNN
+F 1 "-15V" H 750 2400 50  0000 C CNN
+F 2 "" H 750 2250 50  0000 C CNN
+F 3 "" H 750 2250 50  0000 C CNN
+	1    750  2250
+	-1   0    0    1
+$EndComp
+Connection ~ 750  2150
 $Comp
 L R R?
@@
 Wire Wire Line
 	3750 4150 3750 4200
-Wire Wire Line
-	575  10200 3850 10200
-Connection ~ 3375 10200
 $Comp
 L R R?
@@
 	3750 9550 3750 9600
 Wire Wire Line
-	3675 9600 3850 9600
-Wire Wire Line
 	3750 8950 3750 9500
 Connection ~ 3750 9500
 Wire Wire Line
 	3750 1100 3750 1500
-Connection ~ 2225 1100
 Text GLabel 1250 3750 0    60   Input ~ 0
 TECLADO_D0
@@
 Wire Wire Line
 	1250 4050 1900 4050
-Wire Wire Line
-	1075 1550 1075 2625
-Wire Wire Line
-	1075 2625 575  2625
-Wire Wire Line
-	575  2625 575  10200
 Wire Wire Line
 	5450 9500 5250 9500
@@
 	1400 1000 1525 1000
 Wire Wire Line
-	725  775  725  1250
-Connection ~ 1475 775
-Wire Wire Line
-	1075 1250 1075 775
-Connection ~ 1075 775
+	750  800  750  1275
 $Comp
 L POT RV?
@@
 POT_VOL_MANUAL
 Wire Wire Line
-	6950 8725 7300 8725
-Wire Wire Line
-	7300 8725 7300 8600
+	7300 8725 6950 8725
+Wire Wire Line
+	7300 8225 7300 8725
 $Comp
 L R R?
@@
 	1    0    0    -1
 $EndComp
+$Comp
+L R R?
+U 1 1 59AE34E7
+P 1100 1400
+F 0 "R?" H 1250 1500 50  0000 C CNN
+F 1 "750" H 1250 1400 50  0000 C CNN
+F 2 "" V 1030 1400 50  0000 C CNN
+F 3 "" H 1100 1400 50  0000 C CNN
+	1    1100 1400
+	-1   0    0    1
+$EndComp
+Wire Wire Line
+	1100 1250 1100 800
+Wire Wire Line
+	1100 1550 1100 2600
+Wire Wire Line
+	1100 2600 600  2600
+Wire Wire Line
+	600  2600 600  9600
+Wire Wire Line
+	600  9600 3850 9600
+$Comp
+L GND #PWR?
+U 1 1 59AF1FBB
+P 3750 10800
+F 0 "#PWR?" H 3750 10550 50  0001 C CNN
+F 1 "GND" H 3750 10650 50  0000 C CNN
+F 2 "" H 3750 10800 50  0000 C CNN
+F 3 "" H 3750 10800 50  0000 C CNN
+	1    3750 10800
+	1    0    0    -1
+$EndComp
+Wire Wire Line
+	3850 9700 3750 9700
+Wire Wire Line
+	3750 9700 3750 10800
+Wire Wire Line
+	3850 9800 3750 9800
+Connection ~ 3750 9800
+Wire Wire Line
+	3850 9900 3750 9900
+Connection ~ 3750 9900
+Wire Wire Line
+	3850 10000 3750 10000
+Connection ~ 3750 10000
+Wire Wire Line
+	3850 10100 3750 10100
+Connection ~ 3750 10100
+Wire Wire Line
+	3850 10200 3750 10200
+Connection ~ 3750 10200
+Wire Wire Line
+	1525 1200 1450 1200
+Wire Wire Line
+	1450 1200 1450 800
+Wire Wire Line
+	2200 800  2200 1100
+Connection ~ 2200 1100
+Wire Wire Line
+	750  800  2000 800
+Connection ~ 1450 800
+Connection ~ 1100 800
+$Comp
+L R R?
+U 1 1 59ADB1C7
+P 7300 8075
+F 0 "R?" H 7200 8125 50  0000 C CNN
+F 1 "100K" H 7150 8025 50  0000 C CNN
+F 2 "" V 7230 8075 50  0000 C CNN
+F 3 "" H 7300 8075 50  0000 C CNN
+	1    7300 8075
+	-1   0    0    1
+$EndComp
+Connection ~ 7300 8600
+$Comp
+L GND #PWR?
+U 1 1 59ADB8CA
+P 7300 7850
+F 0 "#PWR?" H 7300 7600 50  0001 C CNN
+F 1 "GND" H 7175 7850 50  0000 C CNN
+F 2 "" H 7300 7850 50  0000 C CNN
+F 3 "" H 7300 7850 50  0000 C CNN
+	1    7300 7850
+	-1   0    0    1
+$EndComp
+Wire Wire Line
+	7300 7850 7300 7925
 $EndSCHEMATC

Commit message: Actualizacion Doc
Other:
- note added: "ADJ_P6"
Changed lines of the file:
@@
 Wire Wire Line
 	7300 7850 7300 7925
+Text Notes 775  2275 0    60   ~ 12
+ADJ_P6
 $EndSCHEMATC
