File: Nuevos_Modulos/COM/Hw/Formant_V2_COM.sch (KiCad schematic (older format))
At the start: 1 part

Commit message: Actualizacion Documentacion
Parts:
- removed U?: DS1801, symbol DS1801
Changed lines of the file:
@@
 Comment4 ""
 $EndDescr
-$Comp
-L DS1801 U?
-U 1 1 5995BB66
-P 2875 5350
-F 0 "U?" H 2375 5350 60  0000 C CNN
-F 1 "DS1801" H 2775 3850 60  0000 C CNN
-F 2 "" H 2875 5350 60  0001 C CNN
-F 3 "" H 2875 5350 60  0001 C CNN
-	1    2875 5350
-	-1   0    0    -1
-$EndComp
-Text GLabel 4275 5850 2    60   Input ~ 0
-COM_VOL_DATA
-Text GLabel 4275 5750 2    60   Input ~ 0
-COM_VOL_CLOCK
-Text GLabel 4275 5650 2    60   Input ~ 0
-COM_VOL_RESET
-Wire Wire Line
-	4275 5650 3625 5650
-Wire Wire Line
-	4275 5750 3625 5750
-Wire Wire Line
-	4275 5850 3625 5850
 $EndSCHEMATC
