File: Modulos/INTERFACE-TECLADO/Hw/Ver_Analogico/Formant_V2_Teclado.sch (KiCad schematic (older format))
At the start: 133 parts

Commit message: Actualizacion Interfaz Teclado
Parts:
- removed C?: 680nF, symbol C_Small
- removed D?: 1N4148, symbol D
- removed Q? (x4): BF256B, TO-92, symbol BF245B
- removed R? (x3): *12K 1%, symbol R
- removed R?: 1M, symbol R
- added P?: KBV/PRUEBAS, symbol CONN_01X03
- added R?: 100, symbol R
- added RV? (x2): 20K, symbol POT_TRIM
- added U?: LF356, symbol LM741
Connections:
- wire segments 556 -> 557
Other:
- moved on the sheet: 10uF/16v, C?, R?, RV?, U?
