File: Modulos/INTERFACE-TECLADO/Hw/Ver_DAC_12Bits/Formant_V2_Teclado.sch (KiCad schematic (older format))
At the start: 87 parts

Commit message: Actualizacion Interfaz Teclado
Parts:
- removed C?: 680nF, symbol C_Small
- removed C? (x2): 220nF, symbol C_Small
- removed C?: 22nF, symbol C_Small
- removed C? (x2): 100nF, symbol C_Small
- removed D? (x2): 1N4148, symbol D
- removed Q? (x4): BF256B, TO-92, symbol BF245B
- removed R? (x2): 1K, symbol R
- removed R? (x3): *12K 1%, symbol R
- removed R?: 1M, symbol R
- removed R?: 100K, symbol R
- removed R?: 12K, symbol R
- removed R?: 2K2, symbol R
- removed R?: *100K, symbol R
- removed R?: 8K2 1%, symbol R
- removed R?: 270, symbol R
- removed R?: 2K7, symbol R
- removed RV?: 100K, symbol POT_TRIM
- removed RV?: *100K, symbol POT_TRIM
- removed RV? (x2): 10K, symbol POT
- removed RV?: 2K, symbol POT
- removed U? (x4): LM358, symbol LM358
- removed U?: LM723, symbol LM723
- removed U?: TLC7524, symbol TLC7524
- added 20K: POT_TRIM, symbol POT_TRIM
- added C? (x2): 100nF, symbol C_Small
- added R?: 47ohm, symbol R
- added R?: 4K7 1%, symbol R
- added R?: 270, symbol R
- added R?: 2K7 1%, symbol R
- added R?: 1K, symbol R
- added R?: 12K, symbol R
- added R?: 2K2, symbol R
- added RV?: 2K, symbol POT
- added U?: AD7541, symbol AD7541
- added U?: LM723, symbol LM723
- added U?: 74HC595, symbol 74HC595
- added U? (x2): 741, symbol LM741
- added U?: LM741, symbol LM741
- added U?: LF356, symbol LM741
- C?: value 680nF -> 1uF
- R?: value 5K 1% -> 5K6 1%
Connections:
- net labels added: TECLADO_D10, TECLADO_D11, TECLADO_D12, TECLADO_D8, TECLADO_D9
- net labels removed: PUNTO_E, TECLADO_D0
- wire segments 337 -> 310
Other:
- note added: "(*) Resistencia de tolerancia 1%"
- note added: "Ajustar a 4,096V en la\nsalida (Pin 3)"
- note added: "GENERADOR 1V/Oct."
- note added: "H"
- note added: "INTERFACE MIDI Y CONTROL GENERAL"
- note added: "L"
- note removed: "2V3->"
- note removed: "CONVERSOR DAC 1V/Oct."
- note removed: "INTERFACE MIDI"
- note removed: "INTERFACE ORIGINAL"
- moved on the sheet: C?, D?, R?, RV?, U?
