File: Modulos/ADSR/Hw/Formant_V2_ADSR.sch (KiCad schematic (older format))
At the start: 26 parts

Commit message: Actualiazacion HW ADSR
Parts:
- removed 10K, 1MLog (x3): POT, symbol POT
- removed C?: 10uF/16V, symbol CP
- removed C?: 100nF, symbol C
- removed D? (x3): 1N4148, symbol D
- removed R? (x2): 1K, symbol R
- removed R?: 220, symbol R
- removed R? (x2): 470, symbol R
- removed R? (x2): 100K, symbol R
- removed R?: 10K, symbol R
- removed RV?: 20K, symbol POT_TRIM
- removed U? (x2): 4066, symbol 4066
- removed U?: LM358, symbol LM358
- added 10K? (x2), 1MLog? (x6): POT, symbol POT
- added 1N? (x3): D, symbol D
- added C? (x2): 10uF/16V, symbol CP
- added C? (x2): 100nF, symbol C
- added D? (x6): 1N4148, symbol D
- added D? (x2): LED, symbol LED
- added R? (x6): 1K, symbol R
- added R? (x2): 220, symbol R
- added R? (x6): 470, symbol R
- added R? (x2): 10K, symbol R
- added R? (x2): 27K, symbol R
- added RV? (x2): 20K, symbol POT_TRIM
- added U? (x4): 4066, symbol 4066
- added U? (x6): LM358, symbol LM358
Connections:
- net +15V: now also U?.8 (V+), U?.8 (V+), U?.8 (V+), U?.8 (V+), U?.8 (V+), U?.8 (V+)
- net +5V: now also R?.1, R?.1, U?.7 (V-), U?.7 (V-)
- net -15V: now also U?.4 (V-), U?.4 (V-), U?.4 (V-), U?.4 (V-), U?.4 (V-), U?.4 (V-)
- net ADSR_1_ENV: now also R?.1
- net ADSR_1_EOS: now also R?.1
- net GND: now also 10K?.3, 10K?.3, C?.2, C?.2, C?.2, C?.2, D?.2 (A), D?.2 (A), R?.1, R?.1, U?.1 (I/O), U?.11 (I/O), U?.14 (V+), U?.14 (V+), U?.3 (+), U?.4 (I/O), U?.5 (+), U?.8 (I/O)
- net TX: now reaches ARDUINO?.1 (TX)
- net at ARDUINO?.10 (D7): now also U?.12 (ON)
- net at ARDUINO?.19 (A0): now also U?.1, U?.2 (-), U?.3 (+)
- net RX: now reaches ARDUINO?.2 (RX)
- net at ARDUINO?.20 (A1): now also 10K?.2
- net at ARDUINO?.21 (A2): now also U?.5 (+), U?.6 (-), U?.7
- net at ARDUINO?.22 (A3): now also 10K?.2
- net at ARDUINO?.5 (D2): now also 1MLog?.1, 1MLog?.2
- net at ARDUINO?.6 (D3): now also U?.5 (ON)
- net at ARDUINO?.7 (D4): now also U?.13 (ON)
- net at ARDUINO?.8 (D5): now also 1MLog?.1, 1MLog?.2
- net at ARDUINO?.9 (D6): now also U?.6 (ON)
- net at 1N4148.2 (A): now also D?.1 (K), U?.7
- net at 1N4148.1 (K): now also D?.2 (A), R?.1, U?.6 (-)
- new net: 1MLog?.1, 1MLog?.2, U?.10 (O/I)
- new net: 1MLog?.3, R?.1 (x6)
- new net: 1MLog?.1, 1MLog?.2, U?.9 (O/I)
- new net: D?.1 (K), R?.2 (x4)
- new net: 1N?.2 (A), R?.2 (x2)
- new net: 1N?.1 (K), C?.1, D?.1 (K), D?.2 (A), D?.2 (A), U?.5 (+)
- new net: 10K?.1, C?.1, RV?.2, RV?.3 (x2)
- new net: R?.1, R?.2, R?.2, R?.2, U?.7
- new net: R?.2, RV?.1 (x2)
- new net: R?.2, R?.2, U?.6 (-)
- new net: 1MLog?.1, 1MLog?.2, U?.2 (O/I)
- new net: 1MLog?.1, 1MLog?.2, U?.3 (O/I)
- new net: 1N?.1 (K), C?.1, D?.1 (K), D?.2 (A), D?.2 (A), U?.3 (+)
- new net: R?.1, R?.2, R?.2, R?.2, U?.1
- new net: R?.2, R?.2, U?.2 (-)
- new net: 1N?.2 (A), D?.1 (K), U?.1
- new net: 1N?.1 (K), D?.2 (A), R?.1, U?.2 (-)
- new net ADSR_2_ENV: R?.1
- new net ADSR_2_EOS: R?.1
Other:
- note added: "ADSR 1"
- note added: "ADSR 2"
- moved on the sheet: R?

Commit message: Actualizacion ADSR
Parts:
- added R? (x2): 100K, symbol R
Connections:
- net GND: now also R?.2, R?.2
- net at ARDUINO?.13 (D10), SW?.2 (B): now also R?.1
- net at ARDUINO?.14 (D11), SW?.2 (B): now also R?.1
Other:
- moved on the sheet: R?
Changed lines of the file:
@@
 L R R?
 U 1 1 5A06A034
-P 1075 5200
-F 0 "R?" H 950 5250 50  0000 C CNN
-F 1 "100K" H 925 5150 50  0000 C CNN
-F 2 "" V 1005 5200 50  0000 C CNN
-F 3 "" H 1075 5200 50  0000 C CNN
-	1    1075 5200
-	1    0    0    -1
-$EndComp
-Wire Wire Line
-	1075 5050 1075 4975
-Connection ~ 1075 4975
+P 850 6200
+F 0 "R?" H 725 6250 50  0000 C CNN
+F 1 "100K" H 700 6150 50  0000 C CNN
+F 2 "" V 780 6200 50  0000 C CNN
+F 3 "" H 850 6200 50  0000 C CNN
+	1    850  6200
+	1    0    0    -1
+$EndComp
 $Comp
 L GND #PWR?
 U 1 1 5A06A16A
-P 1075 5500
-F 0 "#PWR?" H 1075 5250 50  0001 C CNN
-F 1 "GND" H 1075 5350 50  0001 C CNN
-F 2 "" H 1075 5500 50  0000 C CNN
-F 3 "" H 1075 5500 50  0000 C CNN
-	1    1075 5500
-	1    0    0    -1
-$EndComp
-Wire Wire Line
-	1075 5350 1075 5500
+P 850 6500
+F 0 "#PWR?" H 850 6250 50  0001 C CNN
+F 1 "GND" H 850 6350 50  0001 C CNN
+F 2 "" H 850 6500 50  0000 C CNN
+F 3 "" H 850 6500 50  0000 C CNN
+	1    850  6500
+	1    0    0    -1
+$EndComp
+Wire Wire Line
+	850  6350 850  6500
 $Comp
 L SW_DPDT_x2 SW?
@@
 P 1800 5525
 F 0 "SW?" H 1800 5695 50  0001 C CNN
-F 1 "ADSR_AD_1" H 1800 5725 50  0000 C CNN
+F 1 "ADSR_AD_1" H 2450 5650 50  0000 C CNN
 F 2 "" H 1800 5525 50  0000 C CNN
 F 3 "" H 1800 5525 50  0000 C CNN
@@
 P 1800 5900
 F 0 "SW?" H 1800 6070 50  0001 C CNN
-F 1 "ADSR_AD_2" H 1775 5650 50  0000 C CNN
+F 1 "ADSR_AD_2" H 2450 6025 50  0000 C CNN
 F 2 "" H 1800 5900 50  0000 C CNN
 F 3 "" H 1800 5900 50  0000 C CNN
@@
 	1525 4875 1525 5525
 Wire Wire Line
-	1525 5525 1600 5525
+	1175 5525 1600 5525
 Wire Wire Line
 	1575 4775 1475 4775
 Wire Wire Line
-	1475 4775 1475 5900
+	1475 4775 1475 6050
 Wire Wire Line
 	1475 5900 1600 5900
@@
 	7875 2650 7600 2650
 Connection ~ 7725 2650
+$Comp
+L R R?
+U 1 1 5A48C7E0
+P 1475 6200
+F 0 "R?" H 1350 6250 50  0000 C CNN
+F 1 "100K" H 1325 6150 50  0000 C CNN
+F 2 "" V 1405 6200 50  0000 C CNN
+F 3 "" H 1475 6200 50  0000 C CNN
+	1    1475 6200
+	1    0    0    -1
+$EndComp
+$Comp
+L GND #PWR?
+U 1 1 5A48C7E6
+P 1475 6500
+F 0 "#PWR?" H 1475 6250 50  0001 C CNN
+F 1 "GND" H 1475 6350 50  0001 C CNN
+F 2 "" H 1475 6500 50  0000 C CNN
+F 3 "" H 1475 6500 50  0000 C CNN
+	1    1475 6500
+	1    0    0    -1
+$EndComp
+Wire Wire Line
+	1475 6350 1475 6500
+$Comp
+L R R?
+U 1 1 5A48C976
+P 1175 6200
+F 0 "R?" H 1050 6250 50  0000 C CNN
+F 1 "100K" H 1025 6150 50  0000 C CNN
+F 2 "" V 1105 6200 50  0000 C CNN
+F 3 "" H 1175 6200 50  0000 C CNN
+	1    1175 6200
+	1    0    0    -1
+$EndComp
+$Comp
+L GND #PWR?
+U 1 1 5A48C97C
+P 1175 6500
+F 0 "#PWR?" H 1175 6250 50  0001 C CNN
+F 1 "GND" H 1175 6350 50  0001 C CNN
+F 2 "" H 1175 6500 50  0000 C CNN
+F 3 "" H 1175 6500 50  0000 C CNN
+	1    1175 6500
+	1    0    0    -1
+$EndComp
+Wire Wire Line
+	1175 6350 1175 6500
+Connection ~ 1475 5900
+Wire Wire Line
+	1175 5525 1175 6050
+Connection ~ 1525 5525
+Wire Wire Line
+	850  6050 850  4975
+Connection ~ 850  4975
 $EndSCHEMATC

Commit message: Actualizacion modulos VCO y ADSR
Parts:
- added P?: pulsador para pruebas, symbol CONN_01X02
- R? (x2): value 470 -> 4K7
Connections:
- net +5V: now also P?.1 (P1)
- net GATE: now also P?.2 (P2)
Changed lines of the file:
@@
 Text GLabel 800  4975 0    60   Input ~ 0
 GATE
-Wire Wire Line
-	800  4975 1575 4975
 $Comp
 L R R?
@@
 P 8025 2200
 F 0 "R?" V 8105 2200 50  0000 C CNN
-F 1 "470" V 8025 2200 50  0000 C CNN
+F 1 "4K7" V 8025 2200 50  0000 C CNN
 F 2 "" V 7955 2200 50  0000 C CNN
 F 3 "" H 8025 2200 50  0000 C CNN
@@
 P 7975 5275
 F 0 "R?" V 8055 5275 50  0000 C CNN
-F 1 "470" V 7975 5275 50  0000 C CNN
+F 1 "4K7" V 7975 5275 50  0000 C CNN
 F 2 "" V 7905 5275 50  0000 C CNN
 F 3 "" H 7975 5275 50  0000 C CNN
@@
 	1175 5525 1175 6050
 Connection ~ 1525 5525
-Wire Wire Line
-	850  6050 850  4975
+$Comp
+L CONN_01X02 P?
+U 1 1 5DAD0CD9
+P 650 4650
+F 0 "P?" H 650 4925 50  0000 C CNN
+F 1 "pulsador para pruebas" V 750 4975 50  0000 C CNN
+F 2 "" H 650 4650 50  0000 C CNN
+F 3 "" H 650 4650 50  0000 C CNN
+	1    650  4650
+	-1   0    0    -1
+$EndComp
+Wire Wire Line
+	1575 4975 800  4975
+Wire Wire Line
+	850  4700 850  6050
 Connection ~ 850  4975
+$Comp
+L +5V #PWR?
+U 1 1 5DAD3FDB
+P 1000 4600
+F 0 "#PWR?" H 1000 4450 50  0001 C CNN
+F 1 "+5V" V 975 4800 50  0000 C CNN
+F 2 "" H 1000 4600 50  0000 C CNN
+F 3 "" H 1000 4600 50  0000 C CNN
+	1    1000 4600
+	0    1    1    0
+$EndComp
+Wire Wire Line
+	850  4600 1000 4600
 $EndSCHEMATC
