File: Modulos/VCO/Hw/Formant_V2_VCO_CEM3340.sch (KiCad schematic (older format))
At the start: 89 parts

Commit message: Actualizacion modulos VCO y ADSR
Parts:
- removed C?: 1nF, symbol C
- removed D? (x4): 1N4148, symbol D
- removed R?: 12K, symbol R
- removed R?: 10K, symbol R
- removed R?: 100, symbol R
- removed R?: 100K 1%, symbol R
- removed R? (x2): 100K, symbol R
- removed R?: 47K, symbol R
- removed R? (x2): 390, symbol R
- removed R?: 330K, symbol R
- removed RV?: 50K, symbol POT_TRIM
- removed RV?: 100K, symbol POT_TRIM
- removed U? (x4): LM1458, symbol LM358
- added C?: 1nF, symbol C
- added C?: 680nF, symbol C
- added FINE?: 50K LOG, symbol POT
- added P? (x3): BNC, symbol BNC
- added R?: 47K, symbol R
- added R? (x4): 10K, symbol R
- added R?: 120K, symbol R
- added R?: 15K, symbol R
- added R?: 33K, symbol R
- added R?: 100K, symbol R
- added U? (x2): LM741, symbol LM741
- added U? (x2): LM1458, symbol TL072
- C? (x2): value .1uF -> 10nF
- C?: value .1uF -> .22uF
- C?: value 1nF -> 100nF
- D? (x2): value OA91 -> 1N4148
- R: value 330K -> 360K 1%
- R?: value 200K -> 1M
- R?: value 100K 1% -> 3M3 1%
- R?: value 100K 1% -> 100K 0.1%
- R?: value 10K -> 100K
- R?: value 10K -> 330K
- R? (x2): value 470 -> 15K
- R?: value 470 -> 22K
- R? (x2): value 470 -> 10K
- R?: value 15K -> 47K
- R?: value 10K -> 22K
Connections:
- net +5V is gone; now on net -15V: PW.1
- net +15V: now also FINE.3, U?.7 (V+), R?.2, U?.7 (V+), U?.7 (V+), U?.8 (V+); no longer U?.4 (V-)
- net -15V: now also U?.4 (V-), U?.4 (V-), U?.4 (V-), U?.4 (V-); no longer U?.7 (V+)
- net GND: now also PW.3, PWM.3, C?.2, FINE?.1, P?.2 (Ext), P?.2 (Ext), P?.2 (Ext), R?.1, R?.1, R?.2, U?.3 (+)
- net at U?.10 (TRIANGLE_OUT): now also U?.5 (+); no longer C?.1
- net at R.2, R?.1, R?.1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: now also R?.1, R?.1, R?.2
- net at R?.2, U?.4 (PULSE_OUT): now also C?.2, R?.2
- net at R?.1, U?.5 (P.W.M._CONTROL): now also C?.1, R?.2
- net at U?.9 (SOFT_SYNC_INPUT): now also R?.1; no longer C?.1
- net at C?.2: now also FINE?.2
- net at R?.1: now also R?.2, R?.1, U?.2 (-)
- net at R?.1: now also D?.2 (A)
- net at R?.2: now also U?.3 (+)
- net at R?.1: now also R?.1, R?.2, U?.6
- net at R?.2: now also U?.2 (-), U?.6; no longer D?.2 (A)
- net at R?.1, R?.1, R?.1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: now also U?.3 (+), R?.2; no longer U?.2 (-)
- net at R?.2, U?.6: now also R?.1
- net at R?.2: now also U?.2 (-), R?.2; no longer U?.3 (+)
- net at SW?.3 (C): now also C?.1; no longer C?.2
- net at SW?.3 (C): now also C?.1
- net at D?.1 (K), D?.2 (A), R?.1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: now also U?.3 (+)
- net at R?.1, R?.1: now also U?.2 (-)
- net at C?.2, R?.2: now also U?.1
- net at RV?.1, RV?.2: now also C?.2, R?.2, U?.7
- net ECV: no longer names the net of SW?.1 (A)
- net ECV: now also P?.1 (In)
- net PWM: no longer names the net of PWM.1
- net PWM: now also P?.1 (In)
- new net: C?.1, R?.2
- new net: R?.1, R?.1, R?.1, U?.6 (-)
- new net: FINE?.3, P?.1 (In)
Other:
- note added: "EC input"
- note added: "PWM input"
- note removed: "Scale ADJ."
- moved on the sheet: C?, D?, PW, PWM, R?, RV?
